File: pcb_control_esp.sch (EAGLE design)
At the start: 45 parts, among them IC1 AT24CP, IC2 REG1117, IC4 DS3231SN, IC5 74LS595N, K1 HKE, Q1 BC337, Q2 BC337, X1 VIN

Commit message: pindah jalur downloader
Connections:
- net CLK: now also R10.2
- net STB: no longer R10.2
Changed lines of the file:
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@@
 <junction x="-27.94" y="71.12"/>
+</segment>
+<segment>
+<wire x1="15.24" y1="68.58" x2="25.4" y2="68.58" width="0.1524" layer="91"/>
+<pinref part="R10" gate="G$1" pin="2"/>
+<label x="15.24" y="68.58" size="1.778" layer="95" rot="R180" xref="yes"/>
 </segment>
 </net>
@@
 <label x="27.94" y="121.92" size="1.778" layer="95" rot="R180" xref="yes"/>
 </segment>
-<segment>
-<wire x1="22.86" y1="68.58" x2="25.4" y2="68.58" width="0.1524" layer="91"/>
-<pinref part="R10" gate="G$1" pin="2"/>
-<label x="22.86" y="68.58" size="1.778" layer="95" rot="R180" xref="yes"/>
-</segment>
 </net>

Commit message: swap i2c
Connections:
- net SCL: now also SJR1.GPIO5; no longer SJR1.GPIO4
- net SDA: now also SJR1.GPIO4; no longer SJR1.GPIO5
Changed lines of the file:
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@@
 </segment>
 <segment>
-<wire x1="-50.8" y1="73.66" x2="-48.26" y2="73.66" width="0.1524" layer="91"/>
-<label x="-48.26" y="73.66" size="1.778" layer="95" xref="yes"/>
-<pinref part="SJR1" gate="G$1" pin="GPIO4"/>
+<wire x1="-50.8" y1="76.2" x2="-35.56" y2="76.2" width="0.1524" layer="91"/>
+<label x="-35.56" y="76.2" size="1.778" layer="95" xref="yes"/>
+<pinref part="SJR1" gate="G$1" pin="GPIO5"/>
 </segment>
 </net>
@@
 </segment>
 <segment>
-<wire x1="-50.8" y1="76.2" x2="-35.56" y2="76.2" width="0.1524" layer="91"/>
-<pinref part="SJR1" gate="G$1" pin="GPIO5"/>
-<label x="-35.56" y="76.2" size="1.778" layer="95" xref="yes"/>
+<label x="-35.56" y="73.66" size="1.778" layer="95" xref="yes"/>
+<pinref part="SJR1" gate="G$1" pin="GPIO4"/>
+<wire x1="-35.56" y1="73.66" x2="-50.8" y2="73.66" width="0.1524" layer="91"/>
 </segment>
 </net>
